File: kh_obd2_interface.kicad_pcb (KiCad board)
At the start: 2 copper layers, 12 parts, among them J1 OBD2, Q1 CSD18540Q5B, U1 LM74500-Q1, U2 TVS2700DRV, U3 TPSM53602RDA

Commit message: Some layout
Parts:
- added ?: , , F.Cu at (42.2, 28.4)
- added ?: , , F.Cu at (38.9, 28.4)
- added ?: , , F.Cu at (42.2, 27.4)
- added ?: , , F.Cu at (38.9, 27.4)
- added C6: 100nF, Capacitor_SMD:C_0402_1005Metric, F.Cu at (0.94, 4.74)
- added C7: 22uF, Capacitor_SMD:C_1210_3225Metric, F.Cu at (43.1, 43.5)
- added C8: 100nF, Capacitor_SMD:C_0402_1005Metric, F.Cu at (0.94, 6.71)
- C1: value 0.1uF -> 100nF
- C2: value 47uF -> 220uF; footprint Capacitor_SMD:CP_Elec_6.3x5.8 -> Capacitor_SMD:C_Elec_6.3x5.8
- C3: value 0.22uf -> 220nF
- C5: value 220uF -> 47uF
- U3: value TPSM53602RDA -> TPSM33620S5QRDNRQ1; footprint TIParts:Texas_QFN-FCMOD-11-N.MxOmm-P0.5mm_4EP -> TIParts:RDN0011A-MFG
- moved Q1 25.6 mm to (43.9, 17.6), turned to 0 degrees
- moved R1 21.0 mm to (38.8, 19.5), turned to 180 degrees
- moved U2 17.7 mm to (31.9, 19.5), turned to 180 degrees
- moved C5 10.8 mm to (40.5, 26.8), turned to -90 degrees
- moved C4 7.53 mm to (33.9, 23.2), turned to 90 degrees
- moved C1 7.53 mm to (30.2, 36.6)
- moved U3 3.73 mm to (35.8, 26.6), turned to 90 degrees
- moved C2 2.76 mm to (52.9, 17.8)
- moved U1 2.71 mm to (35.7, 19.2)
Connections:
- C4 pad 1: Net-(U3-VCC) -> Net-(U3-MODE/SYNC)
- C5 pad 1: unconnected-(C5-Pad1) -> GND
- C5 pad 2: unconnected-(C5-Pad2) -> +5V
- U3 pad 11: unconnected-(U3-MODE/SYNC-Pad11) -> Net-(U3-MODE/SYNC)
- U3 pad 2: unconnected-(U3-EN-Pad2) -> +12V
- U3 pad 3: unconnected-(U3-VIN-Pad3) -> +12V
- U3 pad 4: Net-(U3-FB) -> +5V
- U3 pad 5: unconnected-(U3-SW-Pad5) -> (no net)
- U3 pad 6: unconnected-(U3-SW-Pad6) -> (no net)
- U3 pad 7: unconnected-(U3-BOOT-Pad7) -> (no net)
- U3 pad 8: Net-(U3-VCC) -> Net-(U3-MODE/SYNC)
- U3 pad 9: Net-(U3-FB) -> +5V
Routing:
- net +BATT_FUSED: track 0.00 -> 7.05 mm
- net Net-(U3-MODE/SYNC): track 0.00 -> 6.21 mm, vias 0 -> 2
- net +5V: track 0.00 -> 5.06 mm, vias 0 -> 1
- net Net-(Q1-G): track 0.00 -> 1.69 mm
- net Net-(U1-GATE): track 0.00 -> 1.44 mm
- added copper zone on B.Cu, net +5V
- added copper zone on F.Cu, net +5V
