File: pcb/mcu.kicad_sch (KiCad schematic)
At the start: 10 parts, among them U1 STM32G0B1RET6

Commit message: connector prep
Connections:
- net DISPLAY.DC renamed MCU_DISPLAY.DC
- net DISPLAY.RST renamed MCU_DISPLAY.RST
- net DISPLAY.SPI_CLK renamed MCU_DISPLAY.SPI_CLK
- net DISPLAY.SPI_CS renamed MCU_DISPLAY.SPI_CS
- net DISPLAY.SPI_MISO renamed MCU_DISPLAY.SPI_MISO
- net DISPLAY.SPI_MOSI renamed MCU_DISPLAY.SPI_MOSI
